File: rpi-power-HAT/dcdchat.kicad_sch (KiCad schematic)
At the start: 35 parts, among them J1 Screw_Terminal_01x02, J2 Screw_Terminal_01x02, J3 Conn_01x04_Male, J4 Conn_01x03_Male, J5 Conn_01x04_Male, P1 Conn_02x20_Odd_Even, Q1 SUD50P10-43L, Q2 DMG2305UX, U1 AP64500, U2 DMMT5401

Commit message: Done changes in 2.12.2024 message
Parts:
- R10: value 3.3k -> 47k
- R8: value 0.15k -> 150ohm
- R9: value 1.65k -> 10k
Connections:
- net +5V: no longer D2.2 (A)
- net +5VD: now also D2.2 (A)
- net GPIO15(UART0_RX): now also R10.1
- net at J5.2 (Pin_2), R9.2: no longer R10.1
Other:
- moved on the sheet: R10, R9
Changed lines of the file:
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@@
   (junction (at 131.445 41.275) (diameter 0) (color 0 0 0 0)
   )
-  (junction (at 244.475 112.395) (diameter 0) (color 0 0 0 0)
-  )
   (junction (at 31.75 133.985) (diameter 0) (color 0 0 0 0)
   )
@@
   (junction (at 31.75 151.765) (diameter 0) (color 0 0 0 0)
   )
+  (junction (at 237.49 112.395) (diameter 0) (color 0 0 0 0)
+  )
   (junction (at 182.88 56.515) (diameter 0) (color 0 0 0 0)
   )
@@
     (stroke (width 0) (type default) (color 0 0 0 0))
   )
-  (wire (pts (xy 244.475 112.395) (xy 268.605 112.395))
-    (stroke (width 0) (type default) (color 0 0 0 0))
-  )
   (polyline (pts (xy 233.045 17.78) (xy 233.045 80.01))
     (stroke (width 0) (type default) (color 0 0 0 0))
@@
     (stroke (width 0) (type default) (color 0 0 0 0))
   )
-  (wire (pts (xy 240.665 112.395) (xy 244.475 112.395))
-    (stroke (width 0) (type default) (color 0 0 0 0))
-  )
   (wire (pts (xy 50.8 103.505) (xy 58.42 103.505))
     (stroke (width 0) (type default) (color 0 0 0 0))
@@
     (stroke (width 0) (type default) (color 0 0 0 0))
   )
+  (wire (pts (xy 252.73 112.395) (xy 268.605 112.395))
+    (stroke (width 0) (type default) (color 0 0 0 0))
+  )
   (wire (pts (xy 50.8 139.065) (xy 58.42 139.065))
     (stroke (width 0) (type default) (color 0 0 0 0))
@@
     (stroke (width 0) (type default) (color 0 0 0 0))
   )
+  (wire (pts (xy 231.775 112.395) (xy 237.49 112.395))
+    (stroke (width 0) (type default) (color 0 0 0 0))
+  )
   (wire (pts (xy 99.695 46.355) (xy 99.695 45.085))
     (stroke (width 0) (type default) (color 0 0 0 0))
@@
     (stroke (width 0) (type default) (color 0 0 0 0))
   )
-  (wire (pts (xy 244.475 112.395) (xy 244.475 114.935))
+  (wire (pts (xy 237.49 112.395) (xy 237.49 114.935))
     (stroke (width 0) (type default) (color 0 0 0 0))
   )
@@
     (stroke (width 0) (type default) (color 0 0 0 0))
   )
+  (wire (pts (xy 237.49 112.395) (xy 245.11 112.395))
+    (stroke (width 0) (type default) (color 0 0 0 0))
+  )
   (polyline (pts (xy 282.575 139.7) (xy 282.575 165.1))
     (stroke (width 0) (type default) (color 0 0 0 0))
@@
     (stroke (width 0) (type default) (color 0 0 0 0))
   )
-  (wire (pts (xy 244.475 122.555) (xy 244.475 124.46))
+  (wire (pts (xy 237.49 122.555) (xy 237.49 124.46))
     (stroke (width 0) (type default) (color 0 0 0 0))
   )
@@
     (stroke (width 0) (type default) (color 0 0 0 0))
   )
-  (wire (pts (xy 231.775 112.395) (xy 233.045 112.395))
-    (stroke (width 0) (type default) (color 0 0 0 0))
-  )
   (wire (pts (xy 50.8 116.205) (xy 72.39 116.205))
     (stroke (width 0) (type default) (color 0 0 0 0))
@@
     (stroke (width 0) (type default) (color 0 0 0 0))
   )
-  (wire (pts (xy 257.81 109.855) (xy 268.605 109.855))
+  (wire (pts (xy 260.985 109.855) (xy 268.605 109.855))
     (stroke (width 0) (type default) (color 0 0 0 0))
   )
@@
     (effects (font (size 1.27 1.27)) (justify left bottom))
   )
-  (label "GPIO14(UART0_TX)" (at 257.81 109.855 180)
+  (label "GPIO14(UART0_TX)" (at 260.985 109.855 180)
     (effects (font (size 1.27 1.27)) (justify right bottom))
   )
@@
     (pin "2")
   )
-  (symbol (lib_id "Device:R") (at 244.475 118.745 0) (unit 1)
-    (in_bom yes) (on_board yes) (fields_autoplaced)
-    (property "Reference" "R10" (id 0) (at 246.38 117.4749 0)
-      (effects (font (size 1.27 1.27)) (justify left))
-    )
-    (property "Value" "3.3k" (id 1) (at 246.38 120.0149 0)
-      (effects (font (size 1.27 1.27)) (justify left))
-    )
-    (property "Footprint" "" (id 2) (at 242.697 118.745 90)
-      (effects (font (size 1.27 1.27)) hide)
-    )
-    (property "Datasheet" "~" (id 3) (at 244.475 118.745 0)
-      (effects (font (size 1.27 1.27)) hide)
-    )
-    (pin "1")
-    (pin "2")
-  )
-  (symbol (lib_id "power:+5V") (at 218.44 34.925 0) (unit 1)
-    (in_bom yes) (on_board yes) (fields_autoplaced)
-    (property "Reference" "#PWR020" (id 0) (at 218.44 38.735 0)
-      (effects (font (size 1.27 1.27)) hide)
-    )
-    (property "Value" "+5V" (id 1) (at 218.44 29.21 0))
-    (property "Footprint" "" (id 2) (at 218.44 34.925 0)
-      (effects (font (size 1.27 1.27)) hide)
-    )
-    (property "Datasheet" "" (id 3) (at 218.44 34.925 0)
-      (effects (font (size 1.27 1.27)) hide)
-    )
-    (pin "1")
+  (symbol (lib_id "Device:R") (at 237.49 118.745 0) (unit 1)
+    (in_bom yes) (on_board yes) (fields_autoplaced)
+    (property "Reference" "R10" (id 0) (at 240.03 117.4749 0)
+      (effects (font (size 1.27 1.27)) (justify left))
+    )
+    (property "Value" "47k" (id 1) (at 240.03 120.0149 0)
+      (effects (font (size 1.27 1.27)) (justify left))
+    )
+    (property "Footprint" "" (id 2) (at 235.712 118.745 90)
+      (effects (font (size 1.27 1.27)) hide)
+    )
+    (property "Datasheet" "~" (id 3) (at 237.49 118.745 0)
+      (effects (font (size 1.27 1.27)) hide)
+    )
+    (pin "1")
+    (pin "2")
   )
   (symbol (lib_id "Device:L") (at 90.805 37.465 90) (unit 1)
@@
     (pin "1")
   )
-  (symbol (lib_id "power:GND") (at 244.475 124.46 0) (unit 1)
-    (in_bom yes) (on_board yes) (fields_autoplaced)
-    (property "Reference" "#PWR022" (id 0) (at 244.475 130.81 0)
-      (effects (font (size 1.27 1.27)) hide)
-    )
-    (property "Value" "GND" (id 1) (at 244.475 128.905 0))
-    (property "Footprint" "" (id 2) (at 244.475 124.46 0)
-      (effects (font (size 1.27 1.27)) hide)
-    )
-    (property "Datasheet" "" (id 3) (at 244.475 124.46 0)
+  (symbol (lib_id "power:GND") (at 237.49 124.46 0) (unit 1)
+    (in_bom yes) (on_board yes) (fields_autoplaced)
+    (property "Reference" "#PWR022" (id 0) (at 237.49 130.81 0)
+      (effects (font (size 1.27 1.27)) hide)
+    )
+    (property "Value" "GND" (id 1) (at 237.49 128.905 0))
+    (property "Footprint" "" (id 2) (at 237.49 124.46 0)
+      (effects (font (size 1.27 1.27)) hide)
+    )
+    (property "Datasheet" "" (id 3) (at 237.49 124.46 0)
       (effects (font (size 1.27 1.27)) hide)
     )
@@
     (pin "1")
   )
+  (symbol (lib_id "power:+5VD") (at 218.44 34.925 0) (unit 1)
+    (in_bom yes) (on_board yes) (fields_autoplaced)
+    (property "Reference" "#PWR?" (id 0) (at 218.44 38.735 0)
+      (effects (font (size 1.27 1.27)) hide)
+    )
+    (property "Value" "+5VD" (id 1) (at 218.44 29.21 0))
+    (property "Footprint" "" (id 2) (at 218.44 34.925 0)
+      (effects (font (size 1.27 1.27)) hide)
+    )
+    (property "Datasheet" "" (id 3) (at 218.44 34.925 0)
+      (effects (font (size 1.27 1.27)) hide)
+    )
+    (pin "1")
+  )
   (symbol (lib_id "Device:C") (at 123.19 46.99 0) (unit 1)
     (in_bom yes) (on_board yes)
@@
     (pin "1")
   )
-  (symbol (lib_id "Device:R") (at 236.855 112.395 90) (unit 1)
-    (in_bom yes) (on_board yes) (fields_autoplaced)
-    (property "Reference" "R9" (id 0) (at 236.855 106.68 90))
-    (property "Value" "1.65k" (id 1) (at 236.855 109.22 90))
-    (property "Footprint" "" (id 2) (at 236.855 114.173 90)
-      (effects (font (size 1.27 1.27)) hide)
-    )
-    (property "Datasheet" "~" (id 3) (at 236.855 112.395 0)
+  (symbol (lib_id "Device:R") (at 248.92 112.395 90) (unit 1)
+    (in_bom yes) (on_board yes)
+    (property "Reference" "R9" (id 0) (at 248.92 114.935 90))
+    (property "Value" "10k" (id 1) (at 248.92 116.84 90))
+    (property "Footprint" "" (id 2) (at 248.92 114.173 90)
+      (effects (font (size 1.27 1.27)) hide)
+    )
+    (property "Datasheet" "~" (id 3) (at 248.92 112.395 0)
       (effects (font (size 1.27 1.27)) hide)
     )
@@
       (effects (font (size 1.27 1.27)) (justify left))
     )
-    (property "Value" "0.15k" (id 1) (at 220.98 57.1499 0)
+    (property "Value" "150ohm" (id 1) (at 220.98 57.1499 0)
       (effects (font (size 1.27 1.27)) (justify left))
     )
@@
       (reference "#PWR019") (unit 1) (value "+5V") (footprint "")
     )
-    (path "/4ef6afdd-9e82-40f7-8a0d-44f9e25f03c3"
-      (reference "#PWR020") (unit 1) (value "+5V") (footprint "")
-    )
     (path "/0117cf9a-e757-4661-8790-0f9372956772"
       (reference "#PWR021") (unit 1) (value "GND") (footprint "")
@@
       (reference "#PWR031") (unit 1) (value "GND") (footprint "")
     )
+    (path "/bd6cccce-3a1e-48d6-b70a-de8708eb7c93"
+      (reference "#PWR?") (unit 1) (value "+5VD") (footprint "")
+    )
     (path "/9f7ecd50-545a-4b9d-b299-0f3c43b09347"
       (reference "C1") (unit 1) (value "10uF") (footprint "")
@@
     )
     (path "/e2ead913-94b1-49c7-87c3-258d4f66f5a2"
-      (reference "R8") (unit 1) (value "0.15k") (footprint "")
+      (reference "R8") (unit 1) (value "150ohm") (footprint "")
     )
     (path "/d504d254-5c7d-4f08-89ac-c6b02453f740"
-      (reference "R9") (unit 1) (value "1.65k") (footprint "")
+      (reference "R9") (unit 1) (value "10k") (footprint "")
     )
     (path "/4d0fd18f-1019-4793-bd56-e85d7835d1ba"
-      (reference "R10") (unit 1) (value "3.3k") (footprint "")
+      (reference "R10") (unit 1) (value "47k") (footprint "")
     )
     (path "/36a6bf3d-05b3-40e0-8cab-2e634f12426b"
