File: rpi-power-HAT/dcdchat.kicad_sch (KiCad schematic)
At the start: 35 parts, among them J1 Screw_Terminal_01x02, J2 Screw_Terminal_01x02, J3 Conn_01x04_Male, J4 Conn_01x03_Male, J5 Conn_01x04_Male, P1 Conn_02x20_Odd_Even, Q1 SUD50P10-43L, Q2 DMG2305UX, U1 AP64500, U2 DMMT5401

Commit message: Replacing components in PCB editor due to 08.12.2024 message
Parts:
- L1: value 3.6uH -> 4.7uH; footprint Inductor_SMD:L_0805_2012Metric -> YSPI0724-4R7M:IND-SMD_L7.3-W6.6_YSPI07XX
- U2: footprint ultralibDMG2305UX:DMG2305UX-7 -> DMMT5401easyeda:SOT-23-6_L2.9-W1.6-P0.95-LS2.8-BR
Changed lines of the file:
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@@
     (in_bom yes) (on_board yes)
     (property "Reference" "L1" (id 0) (at 90.805 32.385 90))
-    (property "Value" "3.6uH" (id 1) (at 90.805 34.925 90))
-    (property "Footprint" "Inductor_SMD:L_0805_2012Metric" (id 2) (at 90.805 37.465 0)
+    (property "Value" "4.7uH" (id 1) (at 90.805 34.925 90))
+    (property "Footprint" "YSPI0724-4R7M:IND-SMD_L7.3-W6.6_YSPI07XX" (id 2) (at 90.805 37.465 0)
       (effects (font (size 1.27 1.27)) hide)
     )
@@
       (effects (font (size 1.27 1.27)) (justify left))
     )
-    (property "Footprint" "ultralibDMG2305UX:DMG2305UX-7" (id 2) (at 184.15 48.895 0)
+    (property "Footprint" "DMMT5401easyeda:SOT-23-6_L2.9-W1.6-P0.95-LS2.8-BR" (id 2) (at 184.15 48.895 0)
       (effects (font (size 1.27 1.27)) hide)
     )
@@
     )
     (path "/5180be94-31b7-4d31-838d-80210a85d008"
-      (reference "L1") (unit 1) (value "3.6uH") (footprint "Inductor_SMD:L_0805_2012Metric")
+      (reference "L1") (unit 1) (value "4.7uH") (footprint "YSPI0724-4R7M:IND-SMD_L7.3-W6.6_YSPI07XX")
     )
     (path "/16ce5f48-d337-4b38-81be-b303442c7787"
@@
     )
     (path "/ae3f3061-e9e0-45af-9ffe-084324908309"
-      (reference "U2") (unit 1) (value "DMMT5401") (footprint "ultralibDMG2305UX:DMG2305UX-7")
-    )
-  )
+      (reference "U2") (unit 1) (value "DMMT5401") (footprint "DMMT5401easyeda:SOT-23-6_L2.9-W1.6-P0.95-LS2.8-BR")
+    )
+  )

Commit message: Finalize the PCB layout
Parts:
- C1: footprint Capacitor_SMD:C_0805_2012Metric -> Capacitor_SMD:C_2220_5750Metric; LCSC (none) -> C13585
- C2: LCSC (none) -> C2918070
- C3: LCSC (none) -> C28233
- C4: value 39.8pF -> 39pF; LCSC (none) -> C576897
- C5: value OPEN -> 47pF; LCSC (none) -> C113821
- C6, C7, C8: footprint Capacitor_SMD:C_0805_2012Metric -> Capacitor_SMD:C_2220_5750Metric; LCSC (none) -> C784103
- D1: LCSC (none) -> C42387343
- D2: LCSC (none) -> C5875740
- J1, J2: LCSC (none) -> C709041
- J3, J5: LCSC (none) -> C131334
- J4: LCSC (none) -> C131339
- L1: LCSC (none) -> C22463813
- Q1: value SUD50P10-43L -> SUD50P10-43L-TP; LCSC (none) -> C41408040
- Q2: LCSC (none) -> C508197
- R1, R10, R7: LCSC (none) -> C2989281
- R2: LCSC (none) -> C728645
- R3: LCSC (none) -> C865809
- R4: value 119k -> 120k; LCSC (none) -> C865161
- R5: LCSC (none) -> C2692772
- R6, R9: LCSC (none) -> C110775
- R8: LCSC (none) -> C513734
- U1: LCSC (none) -> C2070920
- U2: LCSC (none) -> C154733
Connections:
- net GND: now also J2.2 (Pin_2); no longer J2.1 (Pin_1)
- net VCC: now also J2.1 (Pin_1); no longer J2.2 (Pin_2)
Other:
- note added: "GPIO Connector"
- note removed: "GPIO Connector (named due to https://pinout.xyz/)"
- moved on the sheet: C2, R3
