File: rpi-power-HAT/_autosave-dcdchat.kicad_sch (KiCad schematic)
At the start: 35 parts, among them J1 Screw_Terminal_01x02, J2 Screw_Terminal_01x02, J3 Conn_01x04_Male, J4 Conn_01x03_Male, J5 Conn_01x04_Male, P1 Conn_02x20_Odd_Even, Q1 SUD50P10-43L, Q2 DMG2305UX, U1 AP64500, U2 DMMT5401

Commit message: Assigning footprints and placing components in PCB editor
Parts:
- U2: footprint ultralibDMG2305UX:DMG2305UX-7 -> DMMT5401easyeda:SOT-23-6_L2.9-W1.6-P0.95-LS2.8-BR
Changed lines of the file:
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@@
       (effects (font (size 1.27 1.27)) (justify left))
     )
-    (property "Footprint" "ultralibDMG2305UX:DMG2305UX-7" (id 2) (at 184.15 48.895 0)
+    (property "Footprint" "DMMT5401easyeda:SOT-23-6_L2.9-W1.6-P0.95-LS2.8-BR" (id 2) (at 184.15 48.895 0)
       (effects (font (size 1.27 1.27)) hide)
     )
@@
     )
     (path "/ae3f3061-e9e0-45af-9ffe-084324908309"
-      (reference "U2") (unit 1) (value "DMMT5401") (footprint "ultralibDMG2305UX:DMG2305UX-7")
-    )
-  )
+      (reference "U2") (unit 1) (value "DMMT5401") (footprint "DMMT5401easyeda:SOT-23-6_L2.9-W1.6-P0.95-LS2.8-BR")
+    )
+  )
