File: kicad/dcdchat.kicad_sch (KiCad schematic)
At the start: 35 parts, among them J1 Screw_Terminal_01x02, J2 Screw_Terminal_01x02, J3 Conn_01x04_Male, J4 Conn_01x03_Male, J5 Conn_01x04_Male, P1 Conn_02x20_Odd_Even, Q1 SUD50P10-43L-TP, Q2 DMG2305UX, U1 AP64500, U2 DMMT5401

Commit message: Made improvements to schematic
Parts:
- C6, C7, C8: footprint Capacitor_SMD:C_2220_5750Metric -> Capacitor_SMD:C_1206_3216Metric; LCSC C784103 -> C87996
- J1, J2: footprint JL500-50802G01:CONN-TH_2P-P5.08_JL500-50002G01 -> DB125-2.54-2P-GN:CONN-TH_DB125-2.54-2P-GN; LCSC C709041 -> C918120
- L1: value 4.7uH -> 3.3uH; footprint YSPI0724-4R7M:IND-SMD_L7.3-W6.6_YSPI07XX -> HX_CYA1050-3.3UH:IND-SMD_L11.6-W10.1; LCSC C22463813 -> C7587741
- R10: value 47k -> 20k; LCSC C2989281 -> C469660
