File: kicad/dcdchat.kicad_sch (KiCad schematic)
At the start: 49 parts, among them J1 Screw_Terminal_01x02, J2 Screw_Terminal_01x02, J3 Conn_01x04_Male, J4 Conn_01x03_Male, J5 Conn_01x04_Male, P1 Conn_02x20_Odd_Even, Q1 HSBA100P04_C2987717, Q2 HSBA100P04_C2987717, Q3 MMPQ3904, U1 AP64500, U2 DMMT5401

Commit message: Final improvements
Connections:
- net GPIO16: now also R13.2
- net GPIO22: now also R11.2
- net GPIO23: now also R12.2
- net GPIO26: now also R14.2
- removed net GPIO: R11.2, R12.2, R13.2, R14.2
- no-connect marks 30 -> 26
Changed lines of the file:
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@@
-	)
-	(no_connect
-		(at 16.51 149.86)
 	)
 	(no_connect
@@
 	)
 	(no_connect
-		(at 72.39 147.32)
+		(at 16.51 116.84)
 	)
 	(no_connect
@@
 	)
 	(no_connect
-		(at 72.39 121.92)
+		(at 16.51 142.24)
 	)
 	(no_connect
-		(at 16.51 142.24)
+		(at 16.51 119.38)
 	)
 	(no_connect
@@
 	)
 	(no_connect
-		(at 16.51 121.92)
-	)
-	(no_connect
 		(at 34.29 26.67)
 	)
@@
 	)
 	(no_connect
-		(at 16.51 116.84)
-	)
-	(no_connect
 		(at 16.51 127)
 	)
@@
 	)
 	(no_connect
-		(at 16.51 119.38)
-	)
-	(no_connect
 		(at 72.39 124.46)
 	)
@@
 	(wire
 		(pts
-			(xy 139.7 113.03) (xy 144.78 113.03)
+			(xy 139.7 113.03) (xy 146.05 113.03)
 		)
 		(stroke
@@
 	(wire
 		(pts
-			(xy 139.7 107.95) (xy 144.78 107.95)
+			(xy 139.7 107.95) (xy 146.05 107.95)
 		)
 		(stroke
@@
 	(wire
 		(pts
-			(xy 139.7 118.11) (xy 144.78 118.11)
+			(xy 139.7 118.11) (xy 146.05 118.11)
 		)
 		(stroke
@@
 	(wire
 		(pts
-			(xy 139.7 102.87) (xy 144.78 102.87)
+			(xy 139.7 102.87) (xy 146.05 102.87)
 		)
 		(stroke
@@
 		)
 	)
-	(label "GPIO"
-		(at 144.78 118.11 180)
+	(label "GPIO26"
+		(at 146.05 118.11 180)
 		(effects
 			(font
@@
 		)
 	)
-	(label "GPIO"
-		(at 144.78 113.03 180)
+	(label "GPIO16"
+		(at 146.05 113.03 180)
 		(effects
 			(font
@@
 		)
 	)
-	(label "GPIO"
-		(at 144.78 107.95 180)
+	(label "GPIO23"
+		(at 146.05 107.95 180)
 		(effects
 			(font
@@
 		)
 	)
-	(label "GPIO"
-		(at 144.78 102.87 180)
-		(effects
-			(font
+	(label "GPIO22"
+		(at 146.05 102.87 180)
+		(effects
+			(font

Commit message: Issue #2: Prepare for production
Parts:
- R4: LCSC C865161 -> C103948
Connections:
- net +5V: now also Q2.2 (S), Q2.3 (S)
- net at C1.1, Q1.1 (S), U1.2 (VIN)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: now also Q1.2 (S), Q1.3 (S)
Other:
- note added: "Status LEDs"
- note removed: "Blue LEDs"
- note removed: "I calculated value of R4, C4, R3 using formula in AP64500 doc."
- company: (none) -> KPI Rover
- title: (none) -> RPI Power HAT
Changed lines of the file:
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@@
 	(generator_version "9.0")
 	(paper "A4")
+	(title_block
+		(title "RPI Power HAT")
+		(date "2025-05-25")
+		(rev "1.1")
+		(company "KPI Rover")
+	)
 	(text "USB-A"
 		(exclude_from_sim no)
@@
 		)
 	)
-	(text "Blue LEDs"
+	(text "Status LEDs"
 		(exclude_from_sim no)
 		(at 93.726 89.154 0)
@@
 		)
 	)
-	(text "I calculated value of R4, C4, R3\nusing formula in AP64500 doc. \n"
-		(exclude_from_sim no)
-		(at 109.22 36.83 0)
-		(effects
-			(font
-				(size 1 1)
-				(italic yes)
-			)
-			(justify left bottom)
-		)
+	(junction
+		(at 191.77 27.94)
+		(diameter 0)
+		(color 0 0 0 0)
 	)
 	(junction
@@
 	)
 	(junction
-		(at 110.49 105.41)
+		(at 36.83 29.21)
 		(diameter 0)
 		(color 0 0 0 0)
 	)
 	(junction
-		(at 116.84 45.72)
+		(at 110.49 105.41)
 		(diameter 0)
 		(color 0 0 0 0)
@@
 	)
 	(junction
+		(at 105.41 46.99)
+		(diameter 0)
+		(color 0 0 0 0)
+	)
+	(junction
 		(at 31.75 134.62)
 		(diameter 0)
@@
 	)
 	(junction
+		(at 36.83 26.67)
+		(diameter 0)
+		(color 0 0 0 0)
+	)
+	(junction
 		(at 105.41 38.1)
 		(diameter 0)
@@
 	)
 	(junction
-		(at 105.41 45.72)
-		(diameter 0)
-		(color 0 0 0 0)
-	)
-	(junction
 		(at 189.23 45.085)
 		(diameter 0)
@@
 	)
 	(junction
+		(at 116.84 46.99)
+		(diameter 0)
+		(color 0 0 0 0)
+	)
+	(junction
+		(at 191.77 30.48)
+		(diameter 0)
+		(color 0 0 0 0)
+	)
+	(junction
 		(at 58.42 119.38)
 		(diameter 0)
@@
 	(wire
 		(pts
+			(xy 36.83 26.67) (xy 36.83 29.21)
+		)
+		(stroke
+			(width 0)
+			(type default)
+		)
+	)
+	(wire
+		(pts
 			(xy 50.8 121.92) (xy 72.39 121.92)
 		)
@@
 	(wire
 		(pts
-			(xy 105.41 45.72) (xy 116.84 45.72)
+			(xy 105.41 46.99) (xy 116.84 46.99)
 		)
 		(stroke
@@
 	(wire
 		(pts
+			(xy 116.84 46.99) (xy 116.84 45.72)
+		)
+		(stroke
+			(width 0)
+			(type default)
+		)
+	)
+	(wire
+		(pts
 			(xy 50.8 53.34) (xy 50.8 55.88)
 		)
@@
 	(wire
 		(pts
+			(xy 36.83 29.21) (xy 42.545 29.21)
+		)
+		(stroke
+			(width 0)
+			(type default)
+		)
+	)
+	(wire
+		(pts
 			(xy 50.8 111.76) (xy 72.39 111.76)
 		)
@@
 	(wire
 		(pts
+			(xy 190.5 25.4) (xy 191.77 25.4)
+		)
+		(stroke
+			(width 0)
+			(type default)
+		)
+	)
+	(wire
+		(pts
 			(xy 190.5 30.48) (xy 191.77 30.48)
 		)
@@
 	(wire
 		(pts
+			(xy 36.83 24.13) (xy 36.83 26.67)
+		)
+		(stroke
+			(width 0)
+			(type default)
+		)
+	)
+	(wire
+		(pts
 			(xy 58.42 127) (xy 58.42 139.7)
 		)
@@
 	(wire
 		(pts
-			(xy 116.84 45.72) (xy 116.84 48.26)
-		)
-		(stroke
-			(width 0)
-			(type default)
-		)
-	)
-	(wire
-		(pts
 			(xy 16.51 149.86) (xy 38.1 149.86)
 		)
@@
 	(wire
 		(pts
+			(xy 116.84 46.99) (xy 116.84 48.26)
+		)
+		(stroke
+			(width 0)
+			(type default)
+		)
+	)
+	(wire
+		(pts
 			(xy 16.51 142.24) (xy 38.1 142.24)
 		)
@@
 	(wire
 		(pts
+			(xy 34.29 26.67) (xy 36.83 26.67)
+		)
+		(stroke
+			(width 0)
+			(type default)
+		)
+	)
+	(wire
+		(pts
 			(xy 237.49 122.555) (xy 237.49 124.46)
 		)
@@
 	(wire
 		(pts
+			(xy 191.77 25.4) (xy 191.77 27.94)
+		)
+		(stroke
+			(width 0)
+			(type default)
+		)
+	)
+	(wire
+		(pts
 			(xy 266.7 148.59) (xy 258.445 148.59)
 		)
@@
 	(wire
 		(pts
-			(xy 34.29 29.21) (xy 42.545 29.21)
+			(xy 34.29 29.21) (xy 36.83 29.21)
 		)
 		(stroke
@@
 		)
 	)
+	(wire
+		(pts
+			(xy 190.5 27.94) (xy 191.77 27.94)
+		)
+		(stroke
+			(width 0)
+			(type default)
+		)
+	)
 	(polyline
 		(pts
@@
 	(wire
 		(pts
+			(xy 191.77 27.94) (xy 191.77 30.48)
+		)
+		(stroke
+			(width 0)
+			(type default)
+		)
+	)
+	(wire
+		(pts
 			(xy 16.51 111.76) (xy 38.1 111.76)
 		)
@@
 		)
 	)
+	(wire
+		(pts
+			(xy 34.29 24.13) (xy 36.83 24.13)
+		)
+		(stroke
+			(width 0)
+			(type default)
+		)
+	)
 	(label "GPIO12(PWM0)"
 		(at 72.39 142.24 180)
@@
 			)
 		)
-		(property "LCSC" "C865161"
+		(property "LCSC" "C103948"
 			(at 116.84 41.91 0)
 			(effects

Commit message: Issue #4: Made improvements to board
Parts:
- removed Q3: MMPQ3904, MMPQ3904:SOIC-16_L9.9-W3.9-P1.27-LS6.0-BL, symbol MMPQ3904:MMPQ3904
- removed R10: 20k, Resistor_SMD:R_0805_2012Metric, symbol Device:R
- removed R15, R16, R17, R18: 82, Resistor_SMD:R_0805_2012Metric, symbol Device:R
- removed R9: 10k, Resistor_SMD:R_0805_2012Metric, symbol Device:R
- C1: footprint Capacitor_SMD:C_2220_5750Metric -> Capacitor_SMD:C_1206_3216Metric
- J1, J2: footprint DB125-2.54-2P-GN:CONN-TH_DB125-2.54-2P-GN -> DB127V-5.08-2P-GN-S:CONN-TH_2P-P5.08; LCSC C918120 -> C3018698
- R11, R12, R13, R14: value 1k -> 330; LCSC C110774 -> C2989109
- R8: value 150ohm -> 330; LCSC C513734 -> C2989109
- U2: footprint DMMT5401easyeda:SOT-23-6_L2.9-W1.6-P0.95-LS2.8-BR -> Package_TO_SOT_SMD:SOT-23-6
Connections:
- net GND: now also D3.1 (K), D4.1 (K), D5.1 (K), D6.1 (K)
- net GPIO15(UART0_RX): now also J5.2 (Pin_2)
- net at R13.1: now also D5.2 (A)
- net at D4.2 (A): now also R12.1
- net at D3.2 (A): now also R11.1
- net at D6.2 (A): now also R14.1
- net GPIO0(UART1_TX) renamed GPIO0(EEPROM_SDA)
- net GPIO0(EEPROM_SDA): no longer J4.3 (Pin_3)
- net GPIO4(GPCLK0) renamed GPIO4(UART2_TX)
- net GPIO4(UART2_TX): now also J4.3 (Pin_3)
- net GPIO5(UART1_RX) renamed GPIO5(UART2_RX)
Other:
- moved on the sheet: D3, D4, D5, D6, J5, R11

Commit message: Issue #4: Prepare for production
Parts:
- Q1, Q2: LCSC (none) -> C2987717; LCSC Part C2987717 -> (none)
- USB1: LCSC (none) -> C2345; LCSC Part C2345 -> (none)
Changed lines of the file:
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@@
 			)
 		)
-		(property "LCSC Part" "C2987717"
-			(at 44.45 29.21 0)
+		(property "LCSC" "C2987717"
+			(at 29.21 29.21 90)
 			(effects
 				(font
@@
 			)
 		)
-		(property "LCSC Part" "C2987717"
+		(property "LCSC" "C2987717"
 			(at 200.66 30.48 0)
 			(effects
@@
 			)
 		)
-		(property "LCSC Part" "C2345"
+		(property "LCSC" "C2345"
 			(at 218.44 171.45 0)
 			(effects
