File: kicad/dcdchat.kicad_pcb (KiCad board)
At the start: 2 copper layers, 65 x 56.5 mm, 35 parts, among them J1 Screw_Terminal_01x02, J2 Screw_Terminal_01x02, J3 Conn_01x04_Male, J4 Conn_01x03_Male, J5 Conn_01x04_Male, P1 Conn_02x20_Odd_Even, Q1 SUD50P10-43L-TP, Q2 DMG2305UX, U1 AP64500, U2 DMMT5401

Commit message: Final improvements
Parts:
- added D3: BLUE, LED_SMD:LED_0805_2012Metric, F.Cu at (197.1, 66.9)
- added D4: BLUE, LED_SMD:LED_0805_2012Metric, F.Cu at (197.1, 69.0)
- added D5: BLUE, LED_SMD:LED_0805_2012Metric, F.Cu at (197.1, 71.1)
- added D6: BLUE, LED_SMD:LED_0805_2012Metric, F.Cu at (197.1, 73.2)
- added Q3: MMPQ3904, MMPQ3904:SOIC-16_L9.9-W3.9-P1.27-LS6.0-BL, F.Cu at (183.4, 80.4)
- added R11: 1k, Resistor_SMD:R_0805_2012Metric, F.Cu at (175.2, 64.2)
- added R12: 1k, Resistor_SMD:R_0805_2012Metric, F.Cu at (177.3, 64.2)
- added R13: 1k, Resistor_SMD:R_0805_2012Metric, F.Cu at (184.0, 64.2)
- added R14: 1k, Resistor_SMD:R_0805_2012Metric, F.Cu at (186.1, 64.2)
- added R15: 82, Resistor_SMD:R_0805_2012Metric, F.Cu at (193.6, 66.9)
- added R16: 82, Resistor_SMD:R_0805_2012Metric, F.Cu at (193.6, 69.0)
- added R17: 82, Resistor_SMD:R_0805_2012Metric, F.Cu at (193.6, 71.1)
- added R18: 82, Resistor_SMD:R_0805_2012Metric, F.Cu at (193.6, 73.2)
- added USB1: JTJ-USB-AF-08, 902-131A1011D10100:USB-A-TH__USB-AF-90, F.Cu at (192.0, 86.7)
- C6, C7, C8: footprint Capacitor_SMD:C_2220_5750Metric -> Capacitor_SMD:C_1206_3216Metric
- J1, J2: footprint JL500-50802G01:CONN-TH_2P-P5.08_JL500-50002G01 -> DB125-2.54-2P-GN:CONN-TH_DB125-2.54-2P-GN
- L1: value 4.7uH -> 3.3uH; footprint YSPI0724-4R7M:IND-SMD_L7.3-W6.6_YSPI07XX -> HX_CYA1050-3.3UH:IND-SMD_L11.6-W10.1
- Q1: value SUD50P10-43L-TP -> HSBA100P04_C2987717; footprint Package_TO_SOT_SMD:TO-252-2 -> HSBA100P04:DFN-8_L5.7-W5.1-P1.27-LS6.1-BL-1
- Q2: value DMG2305UX -> HSBA100P04_C2987717; footprint ultralibDMG2305UX:DMG2305UX-7 -> HSBA100P04:DFN-8_L5.7-W5.1-P1.27-LS6.1-BL-1
- R10: value 47k -> 20k
- moved D2 49.2 mm to (139.7, 73.0), turned to -90 degrees
- moved R8 45.4 mm to (142.2, 73.0), turned to 90 degrees
- moved C8 8.56 mm to (162.9, 91.5)
- moved C6 7.66 mm to (168.1, 91.5)
- moved Q2 5.14 mm to (154.7, 85.5)
- moved L1 3.34 mm to (175.8, 91.8)
- moved Q1 1.75 mm to (154.2, 107.2), turned to 90 degrees
- moved C7 1.29 mm to (165.5, 91.5)
- moved J1 1.16 mm to (141.5, 68.2)
- moved C5 0.67 mm to (172.7, 108.1)
- moved R4 0.67 mm to (172.7, 106.0)
Connections:
- C1 pad 1: Net-(Q1-S) -> Net-(U1-EN)
- Q1 pad 1: Net-(Q1-G) -> Net-(U1-EN)
- Q1 pad 2: VCC -> unconnected-(Q1-S-Pad2)
- Q1 pad 3: Net-(Q1-S) -> unconnected-(Q1-S-Pad3)
- Q2 pad 1: Net-(U2-C2) -> +5V
- Q2 pad 2: +5V -> unconnected-(Q2-S-Pad2)
- Q2 pad 3: +5VD -> unconnected-(Q2-S-Pad3)
- R7 pad 1: Net-(U2-C2) -> Net-(Q2-G)
- U1 pad 2: Net-(Q1-S) -> Net-(U1-EN)
- U1 pad 3: Net-(Q1-S) -> Net-(U1-EN)
- U2 pad 4: Net-(U2-C2) -> Net-(Q2-G)
Routing:
- net +5V: track 98.3 -> 182.8 mm
- net Net-(D3-K): track 0.00 -> 30.3 mm
- net GND: track 9.86 -> 37.5 mm
- net Net-(D4-K): track 0.00 -> 25.4 mm
- net Net-(Q3-B1): track 0.00 -> 21.1 mm
- net Net-(D5-K): track 0.00 -> 20.1 mm
- net Net-(Q3-B2): track 0.00 -> 17.9 mm
- net /GPIO23: track 0.00 -> 17.6 mm
- net Net-(Q3-B3): track 0.00 -> 16.7 mm
- net Net-(D6-K): track 0.00 -> 15.1 mm
- net Net-(Q3-B4): track 0.00 -> 13.8 mm
- net /GPIO22: track 0.00 -> 13.5 mm
- net Net-(Q2-G): track 0.00 -> 10.7 mm
- net +5VD: track 32.6 -> 43.2 mm, vias 2 -> 4
- net Net-(U1-EN): track 0.00 -> 8.21 mm
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- added copper zone on F.Cu, net Net-(U1-EN)
- removed copper zone on F.Cu, net Net-(Q1-S)
Other:
- outline, holes or cut-outs redrawn
- board text added: "KPI Rover RPI Power HAT Ver. 1.1"
- board text removed: "KPI Rover RPI Power HAT Ver. 1.0"

Commit message: Issue #2: Prepare for production
Parts:
- U2: footprint DMMT5401easyeda:SOT-23-6_L2.9-W1.6-P0.95-LS2.8-BR -> Package_TO_SOT_SMD:SOT-23-6
- moved U2 0.12 mm to (145.5, 86.0), turned to 0 degrees
Connections:
- C1 pad 1: Net-(U1-EN) -> unconnected-(C1-Pad1)
- Q1 pad 1: Net-(U1-EN) -> unconnected-(C1-Pad1)
- Q1 pad 2: unconnected-(Q1-S-Pad2) -> unconnected-(C1-Pad1)
- Q1 pad 3: unconnected-(Q1-S-Pad3) -> unconnected-(C1-Pad1)
- Q2 pad 2: unconnected-(Q2-S-Pad2) -> +5V
- Q2 pad 3: unconnected-(Q2-S-Pad3) -> +5V
- U1 pad 2: Net-(U1-EN) -> unconnected-(C1-Pad1)
- U1 pad 3: Net-(U1-EN) -> unconnected-(C1-Pad1)
Routing:
- net +5V: track 182.8 -> 130.6 mm, vias 6 -> 27
- net GND: track 37.5 -> 20.9 mm, vias 21 -> 76
- net Net-(U1-EN): track 8.21 -> 0.00 mm
- net Net-(Q3-B3): track 16.7 -> 17.6 mm
- net Net-(Q1-G): track 9.48 -> 9.70 mm, vias 0 -> 2
- net VCC: vias 20 -> 36
- added copper zone on B.Cu, net +5V
- added copper zone on F.Cu, net +5V
- added copper zone on F.Cu, net unconnected-(C1-Pad1)
- removed copper zone on F.Cu, net Net-(U1-EN)
Other:
- rule solder_mask_min_width: 0.25 -> 0.1

Commit message: Issue #4: Made improvements to board
Parts:
- removed Q3: MMPQ3904, MMPQ3904:SOIC-16_L9.9-W3.9-P1.27-LS6.0-BL
- removed R10: 20k, Resistor_SMD:R_0805_2012Metric
- removed R15, R16, R17, R18: 82, Resistor_SMD:R_0805_2012Metric
- removed R9: 10k, Resistor_SMD:R_0805_2012Metric
- C1: footprint Capacitor_SMD:C_2220_5750Metric -> Capacitor_SMD:C_1206_3216Metric
- J1, J2: footprint DB125-2.54-2P-GN:CONN-TH_DB125-2.54-2P-GN -> DB127V-5.08-2P-GN-S:CONN-TH_2P-P5.08
- R11, R12, R13, R14: value 1k -> 330
- R8: value 150ohm -> 330
- moved D2 7.56 mm to (143.8, 79.3)
- moved R8 7.56 mm to (146.4, 79.3)
- moved D3 6.72 mm to (197.5, 73.6)
- moved D6 6.22 mm to (197.5, 67.0)
- moved D4 2.45 mm to (197.5, 71.4)
- moved D5 1.96 mm to (197.5, 69.2)
- moved C1 0.63 mm to (158.2, 99.3)
Connections:
- net /GPIO5(UART1_RX) renamed /GPIO5(UART2_RX)
- D3 pad 1: Net-(D3-K) -> GND
- D4 pad 1: Net-(D4-K) -> GND
- D5 pad 1: Net-(D5-K) -> GND
- D6 pad 1: Net-(D6-K) -> GND
- J4 pad 3: /GPIO0(UART1_TX) -> /GPIO4(UART2_TX)
- J5 pad 2: Net-(J5-Pin_2) -> /GPIO15(UART0_RX)
- P1 pad 27: /GPIO0(UART1_TX) -> /GPIO0(EEPROM_SDA)
- P1 pad 7: /GPIO4(GPCLK0) -> /GPIO4(UART2_TX)
- R11 pad 1: Net-(Q3-B1) -> Net-(D3-A)
- R12 pad 1: Net-(Q3-B2) -> Net-(D4-A)
- R13 pad 1: Net-(Q3-B3) -> Net-(D5-A)
- R14 pad 1: Net-(Q3-B4) -> Net-(D6-A)
Routing:
- net /GPIO4(UART2_TX): track 0.00 -> 36.4 mm
- net +5V: track 130.6 -> 97.3 mm, vias 27 -> 26
- net Net-(D3-K): track 30.3 -> 0.00 mm
- net Net-(D4-K): track 25.4 -> 0.00 mm
- net Net-(D3-A): track 1.65 -> 26.7 mm
- net Net-(D4-A): track 1.65 -> 24.5 mm
- net Net-(Q3-B1): track 21.1 -> 0.00 mm
- net Net-(D5-K): track 20.1 -> 0.00 mm
- net Net-(Q3-B2): track 17.9 -> 0.00 mm
- net Net-(Q3-B3): track 17.6 -> 0.00 mm
- net Net-(D6-K): track 15.1 -> 0.00 mm
- net Net-(Q3-B4): track 13.8 -> 0.00 mm
- net Net-(D5-A): track 1.65 -> 14.4 mm
- net /GPIO0(UART1_TX): track 10.6 -> 0.00 mm
- net Net-(D6-A): track 1.65 -> 11.3 mm
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Other:
- board text added: "KPI Rover RPI Power HAT Ver. 1.2"
- board text removed: "KPI Rover RPI Power HAT Ver. 1.1"
